Commit message: Update ros2 control of hande

File: robotiq_description/urdf/hand_e.ros2_control.xacro (robot description, xacro)
@@ -19,5 +19,5 @@
         </xacro:if>
         <xacro:if value="${sim_gazebo}">
-          <plugin>gz_ros2_control/GzSystem</plugin>
+          <plugin>ign_ros2_control/IgnitionSystem</plugin>
         </xacro:if>
         <xacro:if value="${use_mock_hardware}">
@@ -25,5 +25,5 @@
           <param name="mock_sensor_commands">${mock_sensor_commands}</param>
         </xacro:if>
-        <xacro:unless value="${use_mock_hardware}">
+        <xacro:unless value="${sim_isaac or sim_gazebo or use_mock_hardware}">
           <plugin>robotiq_driver/RobotiqGripperHardwareInterface</plugin>
           <!-- default data from docs - https://blog.robotiq.com/hubfs/support-files/Hand-E_Adaptive_Gripper_ProductSheet_EN_2024-05_WEB.pdf -->

File: robotiq_description/urdf/robotiq_hand_e_macro.urdf.xacro (robot description, xacro)
@@ -84,8 +84,15 @@
             <origin rpy="0 0 0" xyz="${-0.010} ${-0.075/2} ${0.028/2}"/>
             <geometry>
-<!--               <mesh filename="${left_finger_collision}" scale="1.0 1.0 1.0" /> -->
+              <!--               <mesh filename="${left_finger_collision}" scale="1.0 1.0 1.0" /> -->
               <box size="${left_finger_collision_scale}" />
             </geometry>
           </collision>
+          <inertial>
+            <origin xyz="0 0 0" rpy="0 0 0"/>
+            <mass value="0.5"/>
+            <inertia ixx="0.000001" ixy="0.0" ixz="0.0"
+                    iyy="0.000001" iyz="0.0"
+                    izz="0.000001"/>
+          </inertial>
         </link>
         <link name="${prefix}hande_right_finger">
@@ -103,11 +110,26 @@
             <geometry>
               <box size="${right_finger_collision_scale}" />
-<!--               <mesh filename="${right_finger_collision}" scale="1.0 1.0 1.0" /> -->
+              <!--               <mesh filename="${right_finger_collision}" scale="1.0 1.0 1.0" /> -->
             </geometry>
           </collision>
+          <inertial>
+            <origin xyz="0 0 0" rpy="0 0 0"/>
+            <mass value="0.5"/>
+            <inertia ixx="0.000001" ixy="0.0" ixz="0.0"
+                    iyy="0.000001" iyz="0.0"
+                    izz="0.000001"/>
+          </inertial>
       </link>
       <!-- virtual joint to model values coming from the gripper to the geometry - gripper uses
       distance between fingers as command and state values -->
-      <link name="${prefix}hande_finger_distance_link" />
+      <link name="${prefix}hande_finger_distance_link">
+        <inertial>
+          <origin xyz="0 0 0" rpy="0 0 0"/>
+          <mass value="0.5"/>
+          <inertia ixx="0.000001" ixy="0.0" ixz="0.0"
+                  iyy="0.000001" iyz="0.0"
+                  izz="0.000001"/>
+        </inertial>
+      </link>
       <joint name="${prefix}hande_finger_distance" type="prismatic">
         <axis xyz="1 0 0"/>

Commit message: Update left and right mimic controller.

File: robotiq_description/urdf/hand_e.ros2_control.xacro (robot description, xacro)
@@ -13,4 +13,5 @@
     <ros2_control name="${name}" type="system">
       <hardware>
+        <!-- Isaac Sim -->
         <xacro:if value="${sim_isaac}">
           <plugin>topic_based_ros2_control/TopicBasedSystem</plugin>
@@ -18,11 +19,14 @@
           <param name="joint_states_topic">${isaac_joint_states}</param>
         </xacro:if>
-        <xacro:if value="${sim_gazebo}">
-          <plugin>ign_ros2_control/IgnitionSystem</plugin>
+        <!-- Gazebo Sim (not Isaac) -->
+        <xacro:if value="${sim_gazebo and not sim_isaac}">
+          <plugin>gz_ros2_control/GazeboSimSystem</plugin>
         </xacro:if>
-        <xacro:if value="${use_mock_hardware}">
+        <!-- Mock Hardware (not any sim) -->
+        <xacro:if value="${use_mock_hardware and not sim_gazebo and not sim_isaac}">
           <plugin>mock_components/GenericSystem</plugin>
           <param name="mock_sensor_commands">${mock_sensor_commands}</param>
         </xacro:if>
+        <!-- Real Hardware (none of the above) -->
         <xacro:unless value="${sim_isaac or sim_gazebo or use_mock_hardware}">
           <plugin>robotiq_driver/RobotiqGripperHardwareInterface</plugin>
@@ -58,4 +62,28 @@
         </command_interface>
       </joint>
+      <!-- <joint name="${prefix}hande_left_finger_joint">
+        <command_interface name="position">
+          <param name="min">0.0</param>
+          <param name="max">0.025</param>
+        </command_interface>
+        <state_interface name="position">
+          <param name="initial_value">0.025</param>
+        </state_interface>
+        <state_interface name="velocity">
+          <param name="initial_value">0.0</param>
+        </state_interface>
+      </joint>
+      <joint name="${prefix}hande_right_finger_joint">
+        <command_interface name="position">
+          <param name="min">0.0</param>
+          <param name="max">0.025</param>
+        </command_interface>
+        <state_interface name="position">
+          <param name="initial_value">0.025</param>
+        </state_interface>
+        <state_interface name="velocity">
+          <param name="initial_value">0.0</param>
+        </state_interface>
+      </joint> -->
       <!-- Only add this with real and mock hardware mode -->
       <xacro:unless value="${sim_gazebo or sim_isaac}">

File: robotiq_description/urdf/robotiq_hand_e_gripper.urdf.xacro (robot description, xacro)
@@ -2,7 +2,9 @@
 <robot xmlns:xacro="http://wiki.ros.org/xacro" name="schunk_gripper">
   <!-- Use this if parameters are set from the launch file, otherwise delete -->
+  <xacro:arg name="parent" default="base_link" />
   <xacro:arg name="prefix" default="" />
   <xacro:arg name="use_mock_hardware" default="false" />
   <xacro:arg name="mock_sensor_commands" default="false" />
+  <xacro:arg name="sim_gazebo" default="false" />
   <xacro:include filename="$(find robotiq_description)/urdf/robotiq_hand_e_macro.urdf.xacro"/>
   <xacro:include filename="$(find robotiq_description)/urdf/hand_e.ros2_control.xacro"/>
@@ -11,10 +13,11 @@
   <!-- Load robot's macro with parameters -->
   <!-- set prefix if multiple robots are used -->
-  <xacro:robotiq_hande prefix="$(arg prefix)" parent="base_link" >
-    <origin xyz="0 0 0" rpy="0 0 0" />          <!-- position robot in the world -->
+  <xacro:robotiq_hande prefix="$(arg prefix)" parent="$(arg parent)" sim_gazebo="$(arg sim_gazebo)" >
+    <origin xyz="0 0 0" rpy="0 0 0" />
   </xacro:robotiq_hande>
   <xacro:robotiq_hande_ros2_control
     name="robotiq_hande"
     prefix="$(arg prefix)"
+    sim_gazebo="$(arg sim_gazebo)"
     use_mock_hardware="$(arg use_mock_hardware)" />
 </robot>

File: robotiq_description/urdf/robotiq_hand_e_macro.urdf.xacro (robot description, xacro)
@@ -6,9 +6,9 @@
     </material>
     <material name="dark">
-      <color rgba=".1 0.1 0.1 1.0"/>
+      <color rgba="0.1 0.1 0.1 1.0"/>
     </material>
     <!-- Gripper macro hand-e -->
     <xacro:macro name="robotiq_hande" params="
-                 prefix parent *origin
+                 prefix parent sim_gazebo *origin
                  left_finger_visual:=default left_finger_collision:=default
                  left_finger_scale:=default left_finger_collision_scale:=default
@@ -61,5 +61,4 @@
               <geometry>
                   <mesh filename="${file_path}/meshes/collision/hande/hand-e.stl" scale="1.0 1.0 1.0"/>
-                  <!--<mesh filename="${file_path}/meshes/collision/hande/hand-e_convex_hull.stl" scale="1.0 1.0 1.0"/>-->
               </geometry>
           </collision>
@@ -82,8 +81,7 @@
           </visual>
           <collision>
-            <origin rpy="0 0 0" xyz="${-0.010} ${-0.075/2} ${0.028/2}"/>
+            <origin rpy="0 0 0" xyz="0 0 0"/>
             <geometry>
-              <!--               <mesh filename="${left_finger_collision}" scale="1.0 1.0 1.0" /> -->
-              <box size="${left_finger_collision_scale}" />
+              <mesh filename="${left_finger_collision}" scale="1.0 1.0 1.0" />
             </geometry>
           </collision>
@@ -107,8 +105,7 @@
           </visual>
           <collision>
-            <origin rpy="0 0 0" xyz="${0.010} ${-0.075/2} ${0.028/2}"/>
+            <origin rpy="0 0 0" xyz="0 0 0"/>
             <geometry>
-              <box size="${right_finger_collision_scale}" />
-              <!--               <mesh filename="${right_finger_collision}" scale="1.0 1.0 1.0" /> -->
+              <mesh filename="${right_finger_collision}" scale="1.0 1.0 1.0" />
             </geometry>
           </collision>
@@ -138,5 +135,5 @@
         <origin rpy="0 0 0" xyz="0 0 0.099"/>
         <axis xyz="1 0 0"/>
-        <limit effort="180" lower="0.0" upper="${gripper_maximal_stroke}" velocity="0.15"/>
+        <limit effort="180" lower="0.0" upper="${gripper_maximal_stroke}" velocity="0.08"/>
       </joint>
       <joint name="${prefix}hande_left_finger_joint" type="prismatic">
@@ -145,6 +142,6 @@
         <child link="${prefix}hande_left_finger"/>
         <axis xyz="-1 0 0"/>
-        <limit effort="180" lower="0" upper="${gripper_maximal_stroke/2}" velocity="0.15"/>
-        <mimic joint="${prefix}hande_finger_distance" multiplier="-0.5" offset="${gripper_maximal_stroke/2}"/>
+        <limit effort="180" lower="0" upper="${gripper_maximal_stroke/2}" velocity="0.08"/>
+        <!-- <mimic joint="${prefix}hande_finger_distance" multiplier="-0.5" offset="${gripper_maximal_stroke/2}"/> -->
       </joint>
       <joint name="${prefix}hande_right_finger_joint" type="prismatic">
@@ -153,6 +150,6 @@
         <child link="${prefix}hande_right_finger"/>
         <axis xyz="1 0 0"/>
-        <limit effort="180" lower="0" upper="${gripper_maximal_stroke/2}" velocity="0.15"/>
-        <mimic joint="${prefix}hande_finger_distance" multiplier="-0.5" offset="${gripper_maximal_stroke/2}"/>
+        <limit effort="180" lower="0" upper="${gripper_maximal_stroke/2}" velocity="0.08"/>
+        <!-- <mimic joint="${prefix}hande_finger_distance" multiplier="-0.5" offset="${gripper_maximal_stroke/2}"/> -->
       </joint>
       <link name="${prefix}tcp_link"/>

Commit message: temp commit

File: robotiq_description/urdf/hand_e.ros2_control.xacro (robot description, xacro)
@@ -73,6 +73,6 @@
           <param name="initial_value">0.0</param>
         </state_interface>
-      </joint>
-      <joint name="${prefix}hande_right_finger_joint">
+      </joint> -->
+      <!-- <joint name="${prefix}hande_right_finger_joint">
         <command_interface name="position">
           <param name="min">0.0</param>

File: robotiq_description/urdf/robotiq_hand_e_macro.urdf.xacro (robot description, xacro)
@@ -143,5 +143,5 @@
         <axis xyz="-1 0 0"/>
         <limit effort="180" lower="0" upper="${gripper_maximal_stroke/2}" velocity="0.08"/>
-        <!-- <mimic joint="${prefix}hande_finger_distance" multiplier="-0.5" offset="${gripper_maximal_stroke/2}"/> -->
+        <mimic joint="${prefix}hande_finger_distance" multiplier="-0.5" offset="${gripper_maximal_stroke/2}"/>
       </joint>
       <joint name="${prefix}hande_right_finger_joint" type="prismatic">
@@ -151,5 +151,5 @@
         <axis xyz="1 0 0"/>
         <limit effort="180" lower="0" upper="${gripper_maximal_stroke/2}" velocity="0.08"/>
-        <!-- <mimic joint="${prefix}hande_finger_distance" multiplier="-0.5" offset="${gripper_maximal_stroke/2}"/> -->
+        <mimic joint="${prefix}hande_finger_distance" multiplier="-0.5" offset="${gripper_maximal_stroke/2}"/>
       </joint>
       <link name="${prefix}tcp_link"/>

Commit message: Change to debug level update hardware interface.

File: robotiq_description/urdf/hand_e.ros2_control.xacro (robot description, xacro)
@@ -62,5 +62,5 @@
         </command_interface>
       </joint>
-      <!-- <joint name="${prefix}hande_left_finger_joint">
+      <joint name="${prefix}hande_left_finger_joint">
         <command_interface name="position">
           <param name="min">0.0</param>
@@ -85,5 +85,5 @@
           <param name="initial_value">0.0</param>
         </state_interface>
-      </joint> -->
+      </joint>
       <!-- Only add this with real and mock hardware mode -->
       <xacro:unless value="${sim_gazebo or sim_isaac}">

Commit message: restore mimic joint.

File: robotiq_description/urdf/hand_e.ros2_control.xacro (robot description, xacro)
@@ -62,28 +62,4 @@
         </command_interface>
       </joint>
-      <joint name="${prefix}hande_left_finger_joint">
-        <command_interface name="position">
-          <param name="min">0.0</param>
-          <param name="max">0.025</param>
-        </command_interface>
-        <state_interface name="position">
-          <param name="initial_value">0.025</param>
-        </state_interface>
-        <state_interface name="velocity">
-          <param name="initial_value">0.0</param>
-        </state_interface>
-      </joint>
-      <joint name="${prefix}hande_right_finger_joint">
-        <command_interface name="position">
-          <param name="min">0.0</param>
-          <param name="max">0.025</param>
-        </command_interface>
-        <state_interface name="position">
-          <param name="initial_value">0.025</param>
-        </state_interface>
-        <state_interface name="velocity">
-          <param name="initial_value">0.0</param>
-        </state_interface>
-      </joint>
       <!-- Only add this with real and mock hardware mode -->
       <xacro:unless value="${sim_gazebo or sim_isaac}">
