Commit message: Restore values.

File: robotiq_description/urdf/robotiq_hand_e_macro.urdf.xacro (robot description, xacro)
@@ -61,4 +61,5 @@
               <geometry>
                   <mesh filename="${file_path}/meshes/collision/hande/hand-e.stl" scale="1.0 1.0 1.0"/>
+                  <!--<mesh filename="${file_path}/meshes/collision/hande/hand-e_convex_hull.stl" scale="1.0 1.0 1.0"/>-->
               </geometry>
           </collision>
@@ -81,7 +82,8 @@
           </visual>
           <collision>
-            <origin rpy="0 0 0" xyz="0 0 0"/>
+            <origin rpy="0 0 0" xyz="${-0.010} ${-0.075/2} ${0.028/2}"/>
             <geometry>
               <mesh filename="${left_finger_collision}" scale="1.0 1.0 1.0" />
+              <!-- <box size="${left_finger_collision_scale}" /> -->
             </geometry>
           </collision>
@@ -105,7 +107,8 @@
           </visual>
           <collision>
-            <origin rpy="0 0 0" xyz="0 0 0"/>
+            <origin rpy="0 0 0" xyz="${0.010} ${-0.075/2} ${0.028/2}"/>
             <geometry>
               <mesh filename="${right_finger_collision}" scale="1.0 1.0 1.0" />
+              <!-- <box size="${right_finger_collision_scale}" /> -->
             </geometry>
           </collision>
@@ -135,5 +138,5 @@
         <origin rpy="0 0 0" xyz="0 0 0.099"/>
         <axis xyz="1 0 0"/>
-        <limit effort="180" lower="0.0" upper="${gripper_maximal_stroke}" velocity="0.08"/>
+        <limit effort="180" lower="0.0" upper="${gripper_maximal_stroke}" velocity="0.15"/>
       </joint>
       <joint name="${prefix}hande_left_finger_joint" type="prismatic">
@@ -142,5 +145,5 @@
         <child link="${prefix}hande_left_finger"/>
         <axis xyz="-1 0 0"/>
-        <limit effort="180" lower="0" upper="${gripper_maximal_stroke/2}" velocity="0.08"/>
+        <limit effort="180" lower="0" upper="${gripper_maximal_stroke/2}" velocity="0.15"/>
         <mimic joint="${prefix}hande_finger_distance" multiplier="-0.5" offset="${gripper_maximal_stroke/2}"/>
       </joint>
@@ -150,5 +153,5 @@
         <child link="${prefix}hande_right_finger"/>
         <axis xyz="1 0 0"/>
-        <limit effort="180" lower="0" upper="${gripper_maximal_stroke/2}" velocity="0.08"/>
+        <limit effort="180" lower="0" upper="${gripper_maximal_stroke/2}" velocity="0.15"/>
         <mimic joint="${prefix}hande_finger_distance" multiplier="-0.5" offset="${gripper_maximal_stroke/2}"/>
       </joint>

Commit message: updated robot to grip hook properly

File: robotiq_description/urdf/robotiq_hand_e_macro.urdf.xacro (robot description, xacro)
@@ -82,9 +82,26 @@
           </visual>
           <collision>
-            <origin rpy="0 0 0" xyz="${-0.010} ${-0.075/2} ${0.028/2}"/>
+            <origin rpy="0 0 0" xyz="0 0 0"/>
             <geometry>
-              <mesh filename="${left_finger_collision}" scale="1.0 1.0 1.0" />
-              <!-- <box size="${left_finger_collision_scale}" /> -->
+              <mesh filename="${left_finger_visual}" scale="1.0 1.0 1.0" />
             </geometry>
+            <surface>
+              <friction>
+                <ode>
+                  <mu>2.0</mu>
+                  <mu2>2.0</mu2>
+                  <slip1>0.0</slip1>
+                  <slip2>0.0</slip2>
+                </ode>
+              </friction>
+              <contact>
+                <ode>
+                  <kp>1000000.0</kp>
+                  <kd>100.0</kd>
+                  <max_vel>0.01</max_vel>
+                  <min_depth>0.001</min_depth>
+                </ode>
+              </contact>
+            </surface>
           </collision>
           <inertial>
@@ -107,9 +124,25 @@
           </visual>
           <collision>
-            <origin rpy="0 0 0" xyz="${0.010} ${-0.075/2} ${0.028/2}"/>
+            <origin rpy="0 0 0" xyz="0 0 0"/>
             <geometry>
-              <mesh filename="${right_finger_collision}" scale="1.0 1.0 1.0" />
-              <!-- <box size="${right_finger_collision_scale}" /> -->
-            </geometry>
+              <mesh filename="${right_finger_visual}" scale="1.0 1.0 1.0" />            </geometry>
+            <surface>
+              <friction>
+                <ode>
+                  <mu>2.0</mu>
+                  <mu2>2.0</mu2>
+                  <slip1>0.0</slip1>
+                  <slip2>0.0</slip2>
+                </ode>
+              </friction>
+              <contact>
+                <ode>
+                  <kp>1000000.0</kp>
+                  <kd>100.0</kd>
+                  <max_vel>0.01</max_vel>
+                  <min_depth>0.001</min_depth>
+                </ode>
+              </contact>
+            </surface>
           </collision>
           <inertial>
